File: Electronics/Main_PCB/try1.brd (EAGLE design)
At the start: 160 x 100 mm, 58 parts, among them IC1 4051N, J1 USB_MINI-B_SMT, J2 USB_A_SMT_FEMALE, J3 USB_B_PTH, T1 2N3904, X1 MKDSN1,5/2-5,08, X10 MKDSN1,5/4-5,08, X11 MKDSN1,5/4-5,08, X12 MKDSN1,5/4-5,08, X14 MKDSN1,5/4-5,08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

Commit message: try1 finished, HW tests required
Parts:
- removed J3: USB_B_PTH, SparkFun-Connectors:USB-B-PTH
- removed JP5, JP8: JUMPER-SMT_2_NO_SILK_ROUND, SparkFun-Jumpers:SMT-JUMPER_2_NO_SILK_ROUND
- removed JP6: JUMPER-SMT_3_2-NC_PASTE_SILK, SparkFun-Jumpers:SMT-JUMPER_3_2-NC_PASTE_SILK
- added C1, C2, C4: 0.1uF, rcl:C050-024X044
- added C3: 10uF, rcl:E2,5-7
- added J4: 62910416121, Wurth_Connectors_WR-USB:62910416121
- added JP9: (no value), pinhead:1X03
- added PAD4, PAD5, PAD6: (no value), wirepad:3,17/1,3
- R10, R11: device rcl:0204/5 -> rcl:0207/12
- R12, R13: device rcl:0204/7 -> rcl:0207/12
- R2, R3, R4: device rcl:0204/5 -> rcl:0204/7
- moved R12 18.1 mm to (39.4, 76.8)
- moved R13 11.3 mm to (34.9, 76.8)
- moved PAD3 11.0 mm to (20.6, 57.7)
- moved JP7 7.29 mm to (15.3, 65.2), turned to 0 degrees
- moved SG1 6.48 mm to (111.8, 50.8), turned to 180 degrees
- moved PAD2 5.79 mm to (20.6, 47.5)
- moved T1 5.68 mm to (108.0, 39.4)
- moved J1 5.56 mm to (5.08, 30.0)
- moved PAD1 3.95 mm to (20.6, 52.6)
- moved R11 2.84 mm to (134.6, 58.4), turned to 90 degrees
- moved R10 1.80 mm to (130.8, 58.4), turned to 270 degrees
- moved J2 1.42 mm to (3.81, 70.0)
- moved R2 1.27 mm to (72.4, 15.2)
- moved R3 1.27 mm to (62.2, 15.2)
- moved R4 1.27 mm to (67.3, 15.2)
Connections:
- removed net N$14: JP6.1, JP6.2, X15.3, X15.4, X16.2
- removed net N$16: J3.VBUS, JP8.2
- removed net N$9: J1.VBUS, JP5.2
- new net N$8: JP9.1, JP9.2, X15.3, X15.4, X16.2
- new net VBUS: J1.VBUS
- net +3V3: now also C1.1, C2.1, C3.+, C4.1, JP9.3; no longer JP6.3
- net +5V: now also PAD5.1; no longer JP5.1, JP8.1
- net D+: now also J4.3; no longer J3.D+
- net D-: now also J4.2; no longer J3.D-
- net GND: now also C1.2, C2.2, C3.-, C4.2, J4.4, J4.S1, J4.S2, PAD4.1, PAD6.1; no longer J3.GND
Routing:
- net +3V3: track 0.00 -> 352.6 mm, vias 0 -> 8
- net +5V: track 0.00 -> 228.3 mm, vias 0 -> 2
- net N$8: track 0.00 -> 131.7 mm
- net N$14: track 106.4 -> 0.00 mm
- net D+: track 0.00 -> 81.1 mm, vias 0 -> 2
- net D-: track 0.00 -> 63.9 mm
- net GND: track 0.00 -> 29.9 mm, vias 0 -> 6
- net 12V_SENSE: track 79.3 -> 101.6 mm
- net INTERNAL_SERVO_SENSE: track 38.4 -> 29.3 mm
- net N$1: track 66.2 -> 57.8 mm
- net N$2: track 60.1 -> 53.8 mm
- net LED_1: track 39.8 -> 34.9 mm
- net N$3: track 20.3 -> 15.7 mm
- net BUZZER: track 61.2 -> 57.1 mm
- net N$4: track 53.9 -> 49.8 mm
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- added copper zone on layer 16, net GND
Other:
- board size 160 x 100 mm -> 162 x 102 mm
